Commit message: Implementacion de controles

File: urdf/rover_RYCSV.urdf (robot description, URDF)
Before this commit: robot rover_RYCSV, 11 links, 10 joints
Joints:
- joint BogieIzq: type continuous -> fixed

Commit message: First commit

File: urdf/rover_RYCSV.urdf (robot description, URDF)
Before this commit: robot rover_RYCSV, 11 links, 10 joints
Links:
- removed link Bogie_Der
- removed link Bogie_Izq
- removed link Llanta_1
- removed link Llanta_2
- removed link Llanta_3
- removed link Llanta_4
- removed link Llanta_5
- removed link Llanta_6
- removed link Rocker_Der
- removed link Rocker_Izq
- added link Acople_1, mass 0.16994; collision mesh filename=package://rover_RYCSV/meshes/Acople_1.STL; visual mesh filename=package://rover_RYCSV/meshes/Acople_1.STL
- added link Acople_2, mass 0.17034; collision mesh filename=package://rover_RYCSV/meshes/Acople_2.STL; visual mesh filename=package://rover_RYCSV/meshes/Acople_2.STL
- added link Acople_3, mass 0.16994; collision mesh filename=package://rover_RYCSV/meshes/Acople_3.STL; visual mesh filename=package://rover_RYCSV/meshes/Acople_3.STL
- added link Acople_4, mass 0.16994; collision mesh filename=package://rover_RYCSV/meshes/Acople_4.STL; visual mesh filename=package://rover_RYCSV/meshes/Acople_4.STL
- added link Acople_5, mass 0.17034; collision mesh filename=package://rover_RYCSV/meshes/Acople_5.STL; visual mesh filename=package://rover_RYCSV/meshes/Acople_5.STL
- added link Acople_6, mass 0.16994; collision mesh filename=package://rover_RYCSV/meshes/Acople_6.STL; visual mesh filename=package://rover_RYCSV/meshes/Acople_6.STL
- added link Bogie_der, mass 0.051738; collision mesh filename=package://rover_RYCSV/meshes/Bogie_der.STL; visual mesh filename=package://rover_RYCSV/meshes/Bogie_der.STL
- added link Bogie_izq, mass 0.051738; collision mesh filename=package://rover_RYCSV/meshes/Bogie_izq.STL; visual mesh filename=package://rover_RYCSV/meshes/Bogie_izq.STL
- added link Rocker_der, mass 0.1082; collision mesh filename=package://rover_RYCSV/meshes/Rocker_der.STL; visual mesh filename=package://rover_RYCSV/meshes/Rocker_der.STL
- added link Rocker_izq, mass 0.1082; collision mesh filename=package://rover_RYCSV/meshes/Rocker_izq.STL; visual mesh filename=package://rover_RYCSV/meshes/Rocker_izq.STL
- added link Rueda_1, mass 0.31746; collision mesh filename=package://rover_RYCSV/meshes/Rueda_1.STL; visual mesh filename=package://rover_RYCSV/meshes/Rueda_1.STL
- added link Rueda_2, mass 0.31746; collision mesh filename=package://rover_RYCSV/meshes/Rueda_2.STL; visual mesh filename=package://rover_RYCSV/meshes/Rueda_2.STL
- added link Rueda_3, mass 0.31746; collision mesh filename=package://rover_RYCSV/meshes/Rueda_3.STL; visual mesh filename=package://rover_RYCSV/meshes/Rueda_3.STL
- added link Rueda_4, mass 0.31746; collision mesh filename=package://rover_RYCSV/meshes/Rueda_4.STL; visual mesh filename=package://rover_RYCSV/meshes/Rueda_4.STL
- added link Rueda_5, mass 0.31746; collision mesh filename=package://rover_RYCSV/meshes/Rueda_5.STL; visual mesh filename=package://rover_RYCSV/meshes/Rueda_5.STL
- added link Rueda_6, mass 0.31746; collision mesh filename=package://rover_RYCSV/meshes/Rueda_6.STL; visual mesh filename=package://rover_RYCSV/meshes/Rueda_6.STL
- added link base_footprint
- link Caja: mass 0.78839 -> 0.85251
Joints:
- removed joint BogieDer
- removed joint BogieIzq
- removed joint Llanta1
- removed joint Llanta2
- removed joint Llanta3
- removed joint Llanta4
- removed joint Llanta5
- removed joint Llanta6
- removed joint RockerDer
- removed joint RockerIzq
- added joint Acople_1__rueda_1: type revolute, parent Acople_1, child Rueda_1, origin xyz=0 0 -0.011825 rpy=3.0964 -1.5708 0, axis 1 0 0, limit effort=5 velocity=10.0
- added joint Acople_2__rueda_2: type continuous, parent Acople_2, child Rueda_2, origin xyz=0 0 -0.053075 rpy=0.39754 -1.5708 0, axis 1 0 0, limit effort=5 velocity=10.0
- added joint Acople_3__rueda_3: type continuous, parent Acople_3, child Rueda_3, origin xyz=0 0 -0.011825 rpy=2.9847 -1.5708 0, axis 1 0 0, limit effort=5 velocity=10.0
- added joint Acople_4__rueda_4: type continuous, parent Acople_4, child Rueda_4, origin xyz=0 0 -0.011825 rpy=2.596 -1.5708 0, axis 1 0 0, limit effort=5 velocity=10.0
- added joint Acople_5__rueda_5: type continuous, parent Acople_5, child Rueda_5, origin xyz=0 0 -0.053075 rpy=2.744 -1.5708 0, axis 1 0 0, limit effort=5 velocity=10.0
- added joint Acople_6__rueda_6: type continuous, parent Acople_6, child Rueda_6, origin xyz=0 0 -0.011825 rpy=2.5927 -1.5708 0, axis 1 0 0, limit effort=5 velocity=10.0
- added joint Base_caja: type fixed, parent base_footprint, child Caja, origin xyz=0 0 0.24353 rpy=1.5708 0 0, axis 0 0 0
- added joint Bogie_der__acople_4: type continuous, parent Bogie_der, child Acople_4, origin xyz=0.17745 -0.12528 0.021025 rpy=-3.1416 0 -3.1303, axis 0 1 0
- added joint Bogie_der__acople_5: type fixed, parent Bogie_der, child Acople_5, origin xyz=-0.17516 -0.13012 0.0245 rpy=-3.1416 0 2.2097, axis 0 0 0
- added joint Bogie_izq__acople_1: type continuous, parent Bogie_izq, child Acople_1, origin xyz=0.17745 -0.12528 -0.021025 rpy=0 0 0.011289, axis 0 1 0
- added joint Bogie_izq__acople_2: type fixed, parent Bogie_izq, child Acople_2, origin xyz=-0.17516 -0.13012 -0.0185 rpy=0 0 -0.93188, axis 0 0 0
- added joint Caja__rocker_der: type revolute, parent Caja, child Rocker_der, origin xyz=0 0.0533 -0.15991 rpy=3.1416 0 3.1408, axis 0 0 1, limit lower=-3.14159 upper=3.14159 effort=30 velocity=10.0, mimic joint=Caja__rocker_izq multiplier=-1 offset=0
- added joint Caja__rocker_izq: type revolute, parent Caja, child Rocker_izq, origin xyz=0 0.0533 0.28225 rpy=3.1416 0 3.1408, axis 0 0 1, limit lower=-3.14159 upper=3.14159 effort=30 velocity=10.0
- added joint Rocker_der__acople_6: type continuous, parent Rocker_der, child Acople_6, origin xyz=-0.3483 -0.22154 0.020368 rpy=3.1416 0 -3.1416, axis 0 1 0
- added joint Rocker_der__bogie_der: type continuous, parent Rocker_der, child Bogie_der, origin xyz=0.1754 -0.094265 -0.00065699 rpy=0 0 -0.014542, axis 0 0 1
- added joint Rocker_izq__acople_3: type continuous, parent Rocker_izq, child Acople_3, origin xyz=-0.34812 -0.22154 0.0019767 rpy=0 -0.019032 0, axis 0 1 0
- added joint Rocker_izq__bogie_izq: type fixed, parent Rocker_izq, child Bogie_izq, origin xyz=0.175396751230297 -0.0942654690027159 0.0229999999999996 rpy=0 0 -0.0145421781375742, axis 0 0 0

Commit message: Correccion modelo

File: urdf/rover_RYCSV.urdf (robot description, URDF)
Before this commit: robot rover_RYCSV, 18 links, 17 joints
Joints:
- joint Acople_1__rueda_1: limit effort=5 velocity=10.0 -> effort=0.5 velocity=10.0
- joint Acople_2__rueda_2: limit effort=5 velocity=10.0 -> effort=2 velocity=10.0
- joint Acople_3__rueda_3: limit effort=5 velocity=10.0 -> effort=0.5 velocity=10.0
- joint Acople_4__rueda_4: limit effort=5 velocity=10.0 -> effort=2 velocity=10.0
- joint Acople_5__rueda_5: limit effort=5 velocity=10.0 -> effort=0.5 velocity=10.0
- joint Acople_6__rueda_6: limit effort=5 velocity=10.0 -> effort=0.5 velocity=10.0
- joint Caja__rocker_der: mimic joint=Caja__rocker_izq multiplier=-1 offset=0 -> (none)

Commit message: Avance sistema de control de movimiento

File: urdf/rover_RYCSV.urdf (robot description, URDF)
Before this commit: robot rover_RYCSV, 18 links, 17 joints
Joints:
- joint Acople_1__rueda_1: type revolute -> continuous

Commit message: Sistema de movimiento completado

File: urdf/rover_RYCSV.urdf (robot description, URDF)
Before this commit: robot rover_RYCSV, 18 links, 17 joints
Joints:
- joint Bogie_der__acople_4: limit (none) -> effort=0.98 velocity=6.54498
- joint Bogie_izq__acople_1: limit (none) -> effort=0.98 velocity=6.54498
- joint Rocker_der__acople_6: limit (none) -> effort=0.98 velocity=6.54498
- joint Rocker_izq__acople_3: limit (none) -> effort=0.98 velocity=6.54498

Commit message: Correccion modelo movimiento y añadir sensores

File: urdf/rover_RYCSV.urdf (robot description, URDF)
Before this commit: robot rover_RYCSV, 18 links, 17 joints
Links:
- added link Camera, mass 0.025; collision box size=0.01 0.05 0.05; visual box size=0.01 0.05 0.05
- added link GPS, mass 0.005; collision box size=0.025 0.005 0.025; visual box size=0.025 0.005 0.025
- added link IMU, mass 0.005; collision box size=0.025 0.005 0.025; visual box size=0.025 0.005 0.025
- added link Lidar, mass 0.025; collision cylinder length=0.025 radius=0.025; visual cylinder length=0.025 radius=0.025
Joints:
- added joint Caja_GPS: type fixed, parent Caja, child GPS, origin xyz=0.1 0.0025 0.047 rpy=0 0 0, axis 0 0 0
- added joint Caja_IMU: type fixed, parent Caja, child IMU, origin xyz=0 0.0025 0.047 rpy=0 0 0, axis 0 0 0
- added joint Caja_camera: type fixed, parent Caja, child Camera, origin xyz=0.15 0.145 0.047 rpy=0 0 0, axis 0 0 0
- added joint Caja_lidar: type fixed, parent Caja, child Lidar, origin xyz=-0.22 0.0125 0.047 rpy=1.5707 0 0, axis 0 0 0
- joint Rocker_der__bogie_der: limit (none) -> lower=-3.14159 upper=3.14159 effort=30 velocity=10.0; type continuous -> revolute
- joint Rocker_izq__bogie_izq: axis 0 0 0 -> 0 0 1; limit (none) -> lower=-3.14159 upper=3.14159 effort=30 velocity=10.0; type fixed -> revolute
