Commit message: Cambios del spawn de sensores

File: urdf/kinect.gazebo.xacro (robot description, xacro)
@@ -1,5 +1,4 @@
 <?xml version="1.0"?>
 <robot name="kobuki_kinect_sim" xmlns:xacro="http://ros.org/wiki/xacro">
-    <xacro:arg name="kinect_visual" default="true"/>
     <gazebo reference="camera_rgb_frame">
         <sensor name="kinect_camera" type="depth">

File: urdf/lidar.gazebo.xacro (robot description, xacro)
@@ -7,5 +7,5 @@
           <update_rate>20</update_rate>
           <pose>0 0 0 0 0 0</pose>
-          <visualize>true</visualize>
+          <visualize>false</visualize>
           <ray>
             <scan>
@@ -29,5 +29,5 @@
           </ray>
           <plugin name="gazebo_ros_Lidar_controller" filename="libgazebo_ros_laser.so">
-            <topicName>/rover/laser/scan</topicName>
+            <topicName>/rover/lidar</topicName>
             <frameName>Lidar</frameName>
           </plugin>

File: urdf/rover_RYCSV.urdf.xacro (robot description, xacro)
@@ -1,9 +1,9 @@
 <?xml version="1.0" encoding="utf-8"?>
 <robot name="rover_RYCSV" xmlns:xacro="http://ros.org/wiki/xacro">
-  <!--<xacro:include filename="$(find rover_RYCSV)/urdf/camera.gazebo.xacro" />
-  <xacro:include filename="$(find rover_RYCSV)/urdf/lidar.gazebo.xacro" />-->
-  <xacro:include filename="$(find rover_RYCSV)/urdf/kinect.gazebo.xacro" />
-  <xacro:include filename="$(find rover_RYCSV)/urdf/imu.gazebo.xacro" />
-  <xacro:include filename="$(find rover_RYCSV)/urdf/gps.gazebo.xacro" />
+  <xacro:arg name="imu_enable" default="true"/>
+  <xacro:arg name="gps_enable" default="true"/>
+  <!-- Si el sensor kinect esta habilitado entonces la camara y lidar no lo pueden estar-->
+  <xacro:arg name="kinect_enable" default="true"/>
+  <xacro:arg name="camera_and_lidar_enable" default="false"/>
   <link name="base_footprint"/>
   <link
@@ -60,252 +60,4 @@
       xyz="0 0 0" />
   </joint>
-  <!--<link name="Camera">
-    <inertial>
-      <origin
-        xyz="0 0 0"
-        rpy="0 0 0" />
-      <mass
-        value="0.025" />
-      <inertia
-        ixx="0.0001"
-        ixy="0.0"
-        ixz="0.0"
-        iyy="0.0001"
-        iyz="0.0"
-        izz="0.0001" />
-    </inertial>
-    <visual>
-      <origin
-        xyz="0 0 0"
-        rpy="0 0 0" />
-      <geometry>
-        <box size="0.01 0.05 0.05"/>
-      </geometry>
-      <material
-        name="">
-        <color
-          rgba="1 1 1 1" />
-      </material>
-    </visual>
-    <collision>
-      <origin
-        xyz="0 0 0"
-        rpy="0 0 0" />
-      <geometry>
-        <box size="0.01 0.05 0.05"/>
-      </geometry>
-    </collision>
-  </link>
-  <joint
-    name="Caja_camera"
-    type="fixed">
-    <origin
-      xyz="-0.225 0.095 0.047"
-      rpy="-1.570709 3.141592 0" />
-    <parent
-      link="Caja" />
-    <child
-      link="Camera" />
-    <axis
-      xyz="0 0 0" />
-  </joint>
-  <link name="Lidar">
-    <collision>
-      <origin xyz="0 0 0" rpy="0 0 0"/>
-      <geometry>
-    <box size="0.1 0.1 0.1"/>
-      </geometry>
-    </collision>
-    <visual>
-      <origin xyz="0 0 0" rpy="0 0 0"/>
-      <geometry>
-        <mesh filename="package://rover_RYCSV/meshes/hokuyo.dae"/>
-      </geometry>
-    </visual>
-    <inertial>
-      <mass value="1e-5" />
-      <origin xyz="0 0 0" rpy="0 0 0"/>
-      <inertia ixx="1e-6" ixy="0" ixz="0" iyy="1e-6" iyz="0" izz="1e-6" />
-    </inertial>
-  </link>
-  <joint
-    name="Caja_lidar"
-    type="fixed">
-    <origin
-      xyz="-0.225 0.035 0.047"
-      rpy="-1.570709 -3.141592 0" />
-    <parent
-      link="Caja" />
-    <child
-      link="Lidar" />
-    <axis
-      xyz="0 0 0" />
-  </joint>-->
-  <link name="Sensor_kinect">
-    <inertial>
-      <origin
-        xyz="0 0 0"
-        rpy="0 0 0" />
-      <mass
-        value="0.01" />
-      <inertia
-        ixx="0.0001"
-        ixy="0.0"
-        ixz="0.0"
-        iyy="0.0001"
-        iyz="0.0"
-        izz="0.0001" />
-    </inertial>
-    <visual>
-      <origin
-        xyz="0 0 0"
-        rpy="0 0 0" />
-      <geometry>
-        <mesh
-          filename="package://rover_RYCSV/meshes/sensor_kinect.stl"
-          scale= "0.01 0.01 0.01"/>
-      </geometry>
-      <material
-        name="">
-        <color
-          rgba="1 1 1 1" />
-      </material>
-    </visual>
-    <collision>
-      <origin
-        xyz="0 0 0"
-        rpy="0 0 0" />
-      <geometry>
-        <mesh
-          filename="package://rover_RYCSV/meshes/sensor_kinect.stl"
-          scale= "0.01 0.01 0.01"/>
-      </geometry>
-    </collision>
-  </link>
-  <joint
-    name="Caja_kinect"
-    type="fixed">
-    <origin
-      xyz="-0.245 0.035 -0.1"
-      rpy="-1.570709 -1.570709 0" />
-    <parent
-      link="Caja" />
-    <child
-      link="Sensor_kinect" />
-    <axis
-      xyz="0 0 0" />
-  </joint>
-  <link name="camera_depth_frame"/>
-  <joint name="camera_depth_joint" type="fixed">
-    <origin xyz="0.147 0.0 0.02" rpy="0.0 0.0 -1.5707"/>
-    <parent link="Sensor_kinect"/>
-    <child link="camera_depth_frame"/>
-  </joint>
-  <link name="camera_rgb_frame"/>
-  <joint name="camera_rgb_joint" type="fixed">
-    <origin xyz="0.076 0.0 0.02" rpy="0.0 0.0 -1.5707"/>
-    <parent link="Sensor_kinect"/>
-    <child link="camera_rgb_frame"/>
-  </joint>
-  <link name="IMU">
-    <inertial>
-      <origin
-        xyz="0 0 0"
-        rpy="0 0 0" />
-      <mass
-        value="0.005" />
-      <inertia
-        ixx="0.00001"
-        ixy="0.0"
-        ixz="0.0"
-        iyy="0.00001"
-        iyz="0.0"
-        izz="0.00001" />
-    </inertial>
-    <visual>
-      <origin
-        xyz="0 0 0"
-        rpy="0 0 0" />
-      <geometry>
-        <box size="0.025 0.005 0.025"/>
-      </geometry>
-      <material
-        name="">
-        <color
-          rgba="1 1 1 1" />
-      </material>
-    </visual>
-    <collision>
-      <origin
-        xyz="0 0 0"
-        rpy="0 0 0" />
-      <geometry>
-        <box size="0.025 0.005 0.025"/>
-      </geometry>
-    </collision>
-  </link>
-  <joint
-    name="Caja_IMU"
-    type="fixed">
-    <origin
-      xyz="0 0.0025 0.047"
-      rpy="0 0 0" />
-    <parent
-      link="Caja" />
-    <child
-      link="IMU" />
-    <axis
-      xyz="0 0 0" />
-  </joint>
-  <link name="GPS">
-    <inertial>
-      <origin
-        xyz="0 0 0"
-        rpy="0 0 0" />
-      <mass
-        value="0.005" />
-      <inertia
-        ixx="0.00001"
-        ixy="0.0"
-        ixz="0.0"
-        iyy="0.00001"
-        iyz="0.0"
-        izz="0.00001" />
-    </inertial>
-    <visual>
-      <origin
-        xyz="0 0 0"
-        rpy="0 0 0" />
-      <geometry>
-        <box size="0.025 0.005 0.025"/>
-      </geometry>
-      <material
-        name="">
-        <color
-          rgba="1 1 1 1" />
-      </material>
-    </visual>
-    <collision>
-      <origin
-        xyz="0 0 0"
-        rpy="0 0 0" />
-      <geometry>
-        <box size="0.025 0.005 0.025"/>
-      </geometry>
-    </collision>
-  </link>
-  <joint
-    name="Caja_GPS"
-    type="fixed">
-    <origin
-      xyz="0.1 0.0025 0.047"
-      rpy="0 0 0" />
-    <parent
-      link="Caja" />
-    <child
-      link="GPS" />
-    <axis
-      xyz="0 0 0" />
-  </joint>
   <link
     name="Rocker_izq">
@@ -1184,8 +936,10 @@
       effort="0.5" velocity="10.0" />
   </joint>
+  <!-- ____________________________________ACTUADORES____________________________________ -->
+  <!-- MOTORREDUCTORES DE LAS RUEDAS -->
   <transmission name="tranmission_1">
       <type>transmission_interface/SimpleTransmission</type>
       <joint name="Acople_1__rueda_1">
-          <hardwareInterface>hardware_interface/VelocityJointInterface</hardwareInterface> <!-- EffortJointInterface-->
+          <hardwareInterface>hardware_interface/VelocityJointInterface</hardwareInterface>
       </joint>
       <actuator name="left_motor_1">
@@ -1232,5 +986,5 @@
       <type>transmission_interface/SimpleTransmission</type>
       <joint name="Acople_6__rueda_6">
-          <hardwareInterface>hardware_interface/VelocityJointInterface</hardwareInterface><!-- EffortJointInterface-->
+          <hardwareInterface>hardware_interface/VelocityJointInterface</hardwareInterface>
       </joint>
       <actuator name="right_motor_3">
@@ -1238,4 +992,5 @@
       </actuator>
   </transmission>
+  <!-- SERVOMOTORES DE DIRECCION DE LAS LLANTAS -->
   <transmission name="tranmission_7">
       <type>transmission_interface/SimpleTransmission</type>
@@ -1274,4 +1029,5 @@
       </actuator>
   </transmission>
+  <!-- NIVELADORES DE CAJA -->
   <transmission name="tranmission_11">
       <type>transmission_interface/SimpleTransmission</type>
@@ -1292,4 +1048,5 @@
       </actuator>
   </transmission>
+  <!-- ASEGURADORES DE LA UNIONES ENTRE ROCKERS Y BOGIES -->
   <transmission name="tranmission_13">
       <type>transmission_interface/SimpleTransmission</type>
@@ -1310,6 +1067,4 @@
       </actuator>
   </transmission>
-  <!-- Gazebo ROS Plugin-->
-  <!-- Plugin para que Gazebo pueda entender los controladores-->
   <gazebo>
       <plugin name="gazebo_ros_control" filename="libgazebo_ros_control.so">
@@ -1317,3 +1072,268 @@
       </plugin>
    </gazebo>
+  <!-- ____________________________________SENSORES____________________________________ -->
+  <!-- SENSOR KINECT -->
+  <xacro:if value="$(arg kinect_enable)">
+    <xacro:include filename="$(find rover_RYCSV)/urdf/kinect.gazebo.xacro" />
+    <link name="Sensor_kinect">
+      <inertial>
+        <origin
+          xyz="0 0 0"
+          rpy="0 0 0" />
+        <mass
+          value="0.01" />
+        <inertia
+          ixx="0.0001"
+          ixy="0.0"
+          ixz="0.0"
+          iyy="0.0001"
+          iyz="0.0"
+          izz="0.0001" />
+      </inertial>
+      <visual>
+        <origin
+          xyz="0 0 0"
+          rpy="0 0 0" />
+        <geometry>
+          <mesh
+            filename="package://rover_RYCSV/meshes/sensor_kinect.stl"
+            scale= "0.01 0.01 0.01"/>
+        </geometry>
+        <material
+          name="">
+          <color
+            rgba="1 1 1 1" />
+        </material>
+      </visual>
+      <collision>
+        <origin
+          xyz="0 0 0"
+          rpy="0 0 0" />
+        <geometry>
+          <mesh
+            filename="package://rover_RYCSV/meshes/sensor_kinect.stl"
+            scale= "0.01 0.01 0.01"/>
+        </geometry>
+      </collision>
+    </link>
+    <joint
+      name="Caja_kinect"
+      type="fixed">
+      <origin
+        xyz="-0.245 0.035 -0.1"
+        rpy="-1.570709 -1.570709 0" />
+      <parent
+        link="Caja" />
+      <child
+        link="Sensor_kinect" />
+      <axis
+        xyz="0 0 0" />
+    </joint>
+    <link name="camera_depth_frame"/>
+    <joint name="camera_depth_joint" type="fixed">
+      <origin xyz="0.147 0.0 0.02" rpy="0.0 0.0 -1.5707"/>
+      <parent link="Sensor_kinect"/>
+      <child link="camera_depth_frame"/>
+    </joint>
+    <link name="camera_rgb_frame"/>
+    <joint name="camera_rgb_joint" type="fixed">
+      <origin xyz="0.076 0.0 0.02" rpy="0.0 0.0 -1.5707"/>
+      <parent link="Sensor_kinect"/>
+      <child link="camera_rgb_frame"/>
+    </joint>
+  </xacro:if>
+  <!-- CAMARA Y LIDAR -->
+  <xacro:if value="$(arg camera_and_lidar_enable)">
+    <xacro:include filename="$(find rover_RYCSV)/urdf/camera.gazebo.xacro" />
+    <xacro:include filename="$(find rover_RYCSV)/urdf/lidar.gazebo.xacro" />
+    <link name="Camera">
+      <inertial>
+        <origin
+          xyz="0 0 0"
+          rpy="0 0 0" />
+        <mass
+          value="0.025" />
+        <inertia
+          ixx="0.0001"
+          ixy="0.0"
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